File: passive_comp/1Лампа.sch (EAGLE design)
At the start: 18 parts, among them T1 2N2222, T2 2N2222

Commit message: add
add
Parts:
- removed C1, C2: 10uF, SparkFun-Capacitors:10UF-POLAR-RADIAL-2.5MM-25V-20%
- removed LED1, LED2: (no value), adafruit:LED5MM
- removed R: 220, SparkFun-Resistors:100OHM-HORIZ-1/4W-1%
- removed T1, T2: 2N2222, adafruit:2N2222
- added LED_GREEN, LED_RED4, LED_RED5, LED_YELLOW: (no value), adafruit:LED5MM
- added PH1: D1160_12, photo-elements:D1160_12
- R2, R3: value 10k -> 220
- R6: value 220 -> 1k
- R7: value 220 -> 10k
Connections:
- removed net N$10: LED_RED3.A, R7.2
- removed net N$4 (its old number): LED2.A, R4.1
- new net N$9: LED_RED5.A, PH1.2
- net +5V: now also R2.1, R3.1, R4.1; no longer R.1, R2.2, R3.2, R4.2
- net GND: now also LED_GREEN.C, LED_RED4.C, LED_RED5.C, LED_YELLOW.C; no longer T1.E, T2.E
- net N$1: now also LED_RED1.A, R2.2; no longer LED1.A, R1.2
- net N$2: now also LED_YELLOW.A, R3.2; no longer C1.+, LED1.C, T1.C
- net N$3: now also LED_GREEN.A, R4.2; no longer C2.+, LED2.C, T2.C
- net N$5: now also LED_RED3.A, R6.2; no longer C1.-, R2.1, T2.B
- net N$6: now also LED_RED4.A, R7.2; no longer C2.-, R3.1, T1.B
- net N$7: now also R1.2; no longer R.2
- net N$8: now also PH1.1; no longer LED_RED1.A, R6.2
