File: passive_comp/2Светофор.sch (EAGLE design)
At the start: 7 parts

Commit message: add
add
Parts:
- removed SW1: (no value), special:SW_DIP-3
- added S1: (no value), Wurth_Elektronik_Electromechanic_Switch_rev18c:418117170903
Connections:
- net +5V: now also S1.1, S1.2, S1.3; no longer SW1.4, SW1.5, SW1.6
- net N$1: now also S1.5; no longer SW1.2
- net N$4: now also S1.6; no longer SW1.3
- net N$5: now also S1.4; no longer SW1.1
