File: passive_comp/4Конденсатор.sch (EAGLE design)
At the start: 7 parts

Commit message: add
add
Parts:
- removed LED_GREEN, LED_YELLOW: (no value), adafruit:LED5MM
- removed SW1: (no value), special:SW_DIP-3
- added C1, C2, C3, C4: 100uF, SparkFun-Capacitors:100UF-POLAR-RADIAL-2.5MM-25V-20%
- added LED_RED1, LED_RED2: (no value), adafruit:LED5MM
- R2: value 220 -> 10k
Connections:
- removed net N$1: R2.1, SW1.2
- removed net N$10: LED_GREEN.A, R3.2
- removed net N$4: R1.1, SW1.3
- removed net N$5: R3.1, SW1.1
- removed net N$9: LED_YELLOW.A, R2.2
- new net N$2: LED_RED1.A, R2.2
- new net N$3: LED_RED2.A, R3.2
- net +5V: now also C1.+, C2.+, C3.+, C4.+, R1.1, R2.1, R3.1; no longer SW1.4, SW1.5, SW1.6
- net GND: now also C1.-, C2.-, C3.-, C4.-, LED_RED1.C, LED_RED2.C; no longer LED_GREEN.C, LED_YELLOW.C
