File: passive_comp/5Телеграф.sch (EAGLE design)
At the start: 7 parts

Commit message: add
add
Parts:
- removed LED_GREEN, LED_YELLOW: (no value), adafruit:LED5MM
- removed R3: 220, SparkFun-Resistors:100OHM-HORIZ-1/4W-1%
- added C1: 100uF, SparkFun-Capacitors:100UF-POLAR-RADIAL-2.5MM-25V-20%
- added LED_RED1: (no value), adafruit:LED5MM
- added SW2: (no value), adafruit:SWITCH_PUSHBUTTONSOFTTOUCHSMD_SJ
- SW1: device special:SW_DIP-3 -> adafruit:SWITCH_PUSHBUTTONSOFTTOUCHSMD_SJ
Connections:
- removed net N$10: LED_GREEN.A, R3.2
- removed net N$4: R1.1, SW1.3
- removed net N$5: R3.1, SW1.1
- removed net N$9: LED_YELLOW.A, R2.2
- new net N$2: LED_RED1.A, R2.2
- new net N$3: R2.1, SW2.P$2
- net +5V: now also SW1.P$1, SW2.P$1; no longer SW1.4, SW1.5, SW1.6
- net GND: now also C1.-, LED_RED1.C; no longer LED_GREEN.C, LED_YELLOW.C
- net N$1: now also C1.+, R1.1, SW1.P$2; no longer R2.1, SW1.2
