File: activ_copm/Мультивибратор_2.sch (EAGLE design)
At the start: 11 parts, among them Q1 2N2222, Q2 2N2222

Commit message: upd
Parts:
- removed J1: (no value), SparkFun-Connectors:CONN_022.54MM_SCREWTERM
- added C3: 10uF, SparkFun-Capacitors:10UF-POLAR-RADIAL-2.5MM-25V-20%
Connections:
- removed net N$6: C2.-, Q1.B, R3.1
- new net N$7: C2.-, C3.-, Q1.B, R3.1
- net +5V: no longer J1.2
- net GND: no longer J1.1
- net N$3: now also C3.+
Other:
- moved on the sheet: C1, C2, LED1, LED2, Q1, Q2, R1, R2, R3, R4
