File: activ_copm/Мультивибратор_3.sch (EAGLE design)
At the start: 11 parts, among them Q1 2N2222, Q2 2N2222

Commit message: upd
Parts:
- removed J1: (no value), SparkFun-Connectors:CONN_022.54MM_SCREWTERM
- R2: value 10k -> 100k
Connections:
- net +5V: no longer J1.2
- net GND: no longer J1.1
Other:
- moved on the sheet: C1, C2, LED1, LED2, Q1, Q2, R1, R2, R3, R4
